Commit message: fixes

File: nj_220_2_7_description/urdf/nj_220_2_7.xacro (robot description, xacro)
@@ -1,5 +1,5 @@
 <?xml version="1.0" ?>
 <robot xmlns:xacro="http://ros.org/wiki/xacro">
-  <xacro:macro name="nj_220_2_7" params="prefix:='' interface:=hardware_interface/EffortJointInterface">
+  <xacro:macro name="nj_220_2_7" params="prefix:='' interface:=hardware_interface/EffortJointInterface use_fake_hardware">
     <xacro:include filename="$(find nj_220_2_7_description)/urdf/nj_220_2_7_robot.xacro" />
     <xacro:nj_220_2_7_robot prefix="${prefix}"/>
@@ -8,5 +8,6 @@
     <xacro:include filename="$(find nj_220_2_7_description)/urdf/nj_220_2_7_ros2_control.xacro" />
     <xacro:nj_220_2_7_ros2_control prefix="${prefix}"
-                                   name="nj_220_2_7"/>
+                                   name="nj_220_2_7"
+                                   use_fake_hardware="${use_fake_hardware}"/>
   </xacro:macro>
 </robot>

File: nj_220_2_7_description/urdf/nj_220_2_7_ros2_control.xacro (robot description, xacro)
@@ -20,5 +20,5 @@
         </xacro:if>
         <xacro:unless value="${use_fake_hardware}">
-          <plugin>cnr::comau::ComauC5GopenHw</plugin>
+          <plugin>cnr/comau/ComauC5GopenHw</plugin>
           <param name="mqtt_broker_ip">${mqtt_broker_ip}</param>
           <param name="mqtt_client_id">${mqtt_client_id}</param>
