Commit message: fix arg xacro

File: nj-220-27_description/urdf/nj-220-27.xacro (robot description, xacro)
@@ -1,5 +1,15 @@
 <?xml version="1.0" ?>
 <robot xmlns:xacro="http://ros.org/wiki/xacro">
-  <xacro:macro name="nj-220-27" params="prefix:='' transmission_hw_interface:=hardware_interface/EffortJointInterface use_fake_hardware">
+  <xacro:macro name="nj-220-27" params="prefix:=''
+                                        transmission_hw_interface:=hardware_interface/EffortJointInterface use_fake_hardware
+                                        use_fake_hardware:=true
+                                        mqtt_broker_ip:=10.7.7.245
+                                        mqtt_client_id:=comau_c5gopen_hw_mqtt_client
+                                        mqtt_port:=1883
+                                        mqtt_loop_timeout:=1
+                                        topic_fdb_pos_name:=robot/arm1/real_joints_positions
+                                        topic_fdb_vel_name:=robot/arm1/real_joints_velocities
+                                        topic_cmd_name:=robot/arm1/target_joints_trajectory
+                                        read_only:=false">
     <xacro:include filename="$(find nj-220-27_description)/urdf/nj-220-27_robot.xacro" />
     <xacro:nj-220-27_robot prefix="${prefix}"/>
@@ -9,5 +19,13 @@
     <xacro:nj-220-27_ros2_control prefix="${prefix}"
                                   name="nj-220-27"
-                                  use_fake_hardware="${use_fake_hardware}"/>
+                                  use_fake_hardware="${use_fake_hardware}"
+                                  mqtt_broker_ip="${mqtt_broker_ip}"
+                                  mqtt_client_id="${mqtt_client_id}"
+                                  mqtt_port="${mqtt_port}"
+                                  mqtt_loop_timeout="${mqtt_loop_timeout}"
+                                  topic_fdb_pos_name="${topic_fdb_pos_name}"
+                                  topic_fdb_vel_name="${topic_fdb_vel_name}"
+                                  topic_cmd_name="${topic_cmd_name}"
+                                  read_only="${read_only}"/>
   </xacro:macro>
 </robot>

File: nj-220-27_description/urdf/nj-220-27.xacro.urdf (robot description, URDF)
Before this commit: robot nj-220-27, 1 links, 1 joints
Joints:
- removed joint ${prefix}world_to_base_link
- added joint $(arg prefix)world_to_base_link: type fixed, parent world, child $(arg prefix)base_link, origin xyz=0 0 0 rpy=0 0 0

File: nj-220-27_description/urdf/nj-220-27_ros2_control.xacro (robot description, xacro)
@@ -4,5 +4,5 @@
                                                       prefix
                                                       use_fake_hardware:=true
-                                                      mqtt_broker_ip:=10.7.7.246
+                                                      mqtt_broker_ip:=10.7.7.245
                                                       mqtt_client_id:=comau_c5gopen_hw_mqtt_client
                                                       mqtt_port:=1883
